Commit message: Imported upstream version '1.3.0' of 'upstream'

File: sr_description/arm/xacro/lower_arm/shadowarm_lowerarm.urdf.xacro (robot description, xacro)
@@ -24,5 +24,5 @@
     </link>
     <gazebo reference="shadowarm_lowerarm">
-      <material>Gazebo/Grey</material>
+      <material>LightGrey</material>
       <selfCollide>false</selfCollide>
     </gazebo>

File: sr_description/arm/xacro/trunk/shadowarm_trunk.urdf.xacro (robot description, xacro)
@@ -23,5 +23,5 @@
     </link>
     <gazebo reference="shadowarm_trunk">
-      <material>Gazebo/Grey</material>
+      <material>LightGrey</material>
       <selfCollide>false</selfCollide>
     </gazebo>

File: sr_description/arm/xacro/upper_arm/shadowarm_upperarm.urdf.xacro (robot description, xacro)
@@ -23,5 +23,5 @@
     </link>
     <gazebo reference="shadowarm_upperarm">
-      <material>Gazebo/Grey</material>
+      <material>LightGrey</material>
       <selfCollide>false</selfCollide>
     </gazebo>

File: sr_description/hand/xacro/finger/biotac/biotac.urdf.xacro (robot description, xacro)
@@ -29,17 +29,18 @@
     </link>
     <gazebo reference="${link_prefix}adapter">
-      <sensor type="contact" name="${link_prefix}adapter_contact_sensor">
-        <update_rate>100.0</update_rate>
+      <sensor type="contact" name="${link_prefix}adapter_contact" >
+        <always_on>1</always_on>
+        <update_rate>1000.0</update_rate>
         <contact>
-          <collision>${link_prefix}adapter_collision_geom</collision>
+          <collision>${link_prefix}adapter_collision</collision>
+          <topic>${link_prefix}adapter_collision</topic>
         </contact>
         <plugin name="${link_prefix}adapter_gazebo_ros_bumper_controller" filename="libgazebo_ros_bumper.so">
-          <alwaysOn>true</alwaysOn>
-          <frameName>${link_prefix}adapter</frameName>
           <updateRate>100.0</updateRate>
-          <bumperTopicName>${link_prefix}adapter_bumper</bumperTopicName>
+	  <frameName>${link_prefix}adapter</frameName>
+	  <bumperTopicName>contacts/${link_prefix}/adapter</bumperTopicName>
         </plugin>
       </sensor>
-      <material name="LightGrey"/>
+      <material>Gazebo/Grey</material>
     </gazebo>
     <joint name="${joint_prefix}J2" type="revolute">
@@ -90,17 +91,19 @@
     </link>
     <gazebo reference="${link_prefix}biotac">
-      <sensor type="contact" name="${link_prefix}biotac_contact_sensor">
-        <update_rate>100.0</update_rate>
+      <sensor type="contact" name="${link_prefix}biotac_contact" >
+        <always_on>1</always_on>
+        <update_rate>1000.0</update_rate>
         <contact>
-          <collision>${link_prefix}biotac_collision_geom</collision>
+          <collision>${link_prefix}biotac_collision</collision>
+          <topic>${link_prefix}biotac_collision</topic>
         </contact>
         <plugin name="${link_prefix}biotac_gazebo_ros_bumper_controller" filename="libgazebo_ros_bumper.so">
-          <alwaysOn>true</alwaysOn>
-          <frameName>${link_prefix}biotac</frameName>
           <updateRate>100.0</updateRate>
-          <bumperTopicName>${link_prefix}biotac_bumper</bumperTopicName>
+	  <frameName>${link_prefix}biotac</frameName>
+	  <bumperTopicName>contacts/${link_prefix}/biotac</bumperTopicName>
         </plugin>
       </sensor>
-      <material name="BiotacGreen"/>
+      <selfCollide>true</selfCollide>
+      <material>BiotacGreen</material>
     </gazebo>
     <joint name="${joint_prefix}_biotac_joint" type="fixed">

File: sr_description/hand/xacro/finger/biotac/edc_muscle_biotac.urdf.xacro (robot description, xacro)
@@ -29,17 +29,18 @@
     </link>
     <gazebo reference="${link_prefix}adapter">
-      <sensor type="contact" name="${link_prefix}adapter_contact_sensor">
-        <update_rate>100.0</update_rate>
+      <sensor type="contact" name="${link_prefix}adapter_contact" >
+        <always_on>1</always_on>
+        <update_rate>1000.0</update_rate>
         <contact>
-          <collision>${link_prefix}adapter_collision_geom</collision>
+          <collision>${link_prefix}adapter_collision</collision>
+          <topic>${link_prefix}adapter_collision</topic>
         </contact>
         <plugin name="${link_prefix}adapter_gazebo_ros_bumper_controller" filename="libgazebo_ros_bumper.so">
-          <alwaysOn>true</alwaysOn>
-          <frameName>${link_prefix}adapter</frameName>
           <updateRate>100.0</updateRate>
-          <bumperTopicName>${link_prefix}adapter_bumper</bumperTopicName>
+	  <frameName>${link_prefix}adapter</frameName>
+	  <bumperTopicName>contacts/${link_prefix}/adapter</bumperTopicName>
         </plugin>
       </sensor>
-      <material name="LightGrey"/>
+      <material>Gazebo/Grey</material>
     </gazebo>
     <joint name="${joint_prefix}J2" type="revolute">
@@ -90,17 +91,19 @@
     </link>
     <gazebo reference="${link_prefix}biotac">
-      <sensor type="contact" name="${link_prefix}biotac_contact_sensor">
-        <update_rate>100.0</update_rate>
+      <sensor type="contact" name="${link_prefix}biotac_contact" >
+        <always_on>1</always_on>
+        <update_rate>1000.0</update_rate>
         <contact>
-          <collision>${link_prefix}biotac_collision_geom</collision>
+          <collision>${link_prefix}biotac_collision</collision>
+          <topic>${link_prefix}biotac_collision</topic>
         </contact>
         <plugin name="${link_prefix}biotac_gazebo_ros_bumper_controller" filename="libgazebo_ros_bumper.so">
-          <alwaysOn>true</alwaysOn>
-          <frameName>${link_prefix}biotac</frameName>
           <updateRate>100.0</updateRate>
-          <bumperTopicName>${link_prefix}biotac_bumper</bumperTopicName>
+	  <frameName>${link_prefix}biotac</frameName>
+	  <bumperTopicName>contacts/${link_prefix}/biotac</bumperTopicName>
         </plugin>
       </sensor>
-      <material name="BiotacGreen"/>
+      <selfCollide>true</selfCollide>
+      <material>BiotacGreen</material>
     </gazebo>
     <joint name="${joint_prefix}_biotac_joint" type="fixed">

File: sr_description/hand/xacro/finger/distal/distal.urdf.xacro (robot description, xacro)
@@ -30,22 +30,19 @@
     </link>
     <gazebo reference="${link_prefix}distal">
-      <sensor type="contact" name="${link_prefix}distal_contact_sensor">
-        <update_rate>100.0</update_rate>
+      <sensor type="contact" name="${link_prefix}distal_contact" >
+        <always_on>1</always_on>
+        <update_rate>1000.0</update_rate>
         <contact>
-          <collision>${link_prefix}distal_collision_geom</collision>
+          <collision>${link_prefix}distal_collision</collision>
+          <topic>${link_prefix}distal_collision</topic>
         </contact>
         <plugin name="${link_prefix}distal_gazebo_ros_bumper_controller" filename="libgazebo_ros_bumper.so">
-          <alwaysOn>true</alwaysOn>
-          <frameName>${link_prefix}distal</frameName>
           <updateRate>100.0</updateRate>
-          <bumperTopicName>${link_prefix}distal_bumper</bumperTopicName>
+	  <frameName>${link_prefix}distal</frameName>
+	  <bumperTopicName>contacts/${link_prefix}/distal</bumperTopicName>
         </plugin>
       </sensor>
-      <mu1 value="500.0" />
-      <mu2 value="500.0" />
-      <kp  value="10000000.0" />
-      <kd  value="1.0" />
-      <material>Gazebo/Grey</material>
       <selfCollide>true</selfCollide>
+      <material>LightGrey</material>
     </gazebo>
     <joint name="${joint_prefix}J1" type="revolute">
@@ -59,8 +56,8 @@
     </joint>
     <link name="${link_prefix}tip">
-			<inertial>
-				<mass value="0.001" />
-				<inertia  ixx="0.0" ixy="0.0"  ixz="0.0"  iyy="0.0"  iyz="0.0" izz="0.0" />
-  		</inertial>
+      <inertial>
+	<mass value="0.001" />
+	<inertia  ixx="0.0" ixy="0.0"  ixz="0.0"  iyy="0.0"  iyz="0.0" izz="0.0" />
+      </inertial>
     </link>
     <joint name="${joint_prefix}tip" type="fixed">

File: sr_description/hand/xacro/finger/distal/distal_biotac.urdf.xacro (robot description, xacro)
@@ -30,17 +30,19 @@
     </link>
     <gazebo reference="${link_prefix}distal">
-      <sensor type="contact" name="${link_prefix}distal_contact_sensor">
-        <update_rate>100.0</update_rate>
+      <sensor type="contact" name="${link_prefix}distal_contact" >
+        <always_on>1</always_on>
+        <update_rate>1000.0</update_rate>
         <contact>
-          <collision>${link_prefix}distal_collision_geom</collision>
+          <collision>${link_prefix}distal_collision</collision>
+          <topic>${link_prefix}distal_collision</topic>
         </contact>
         <plugin name="${link_prefix}distal_gazebo_ros_bumper_controller" filename="libgazebo_ros_bumper.so">
-          <alwaysOn>true</alwaysOn>
-          <frameName>${link_prefix}distal</frameName>
           <updateRate>100.0</updateRate>
-          <bumperTopicName>${link_prefix}distal_bumper</bumperTopicName>
+	  <frameName>${link_prefix}distal</frameName>
+	  <bumperTopicName>contacts/${link_prefix}/distal</bumperTopicName>
         </plugin>
       </sensor>
-      <material>Gazebo/Grey</material>
+      <selfCollide>true</selfCollide>
+      <material>LightGrey</material>
     </gazebo>
     <joint name="${joint_prefix}J1" type="revolute">

File: sr_description/hand/xacro/finger/distal/distal_ellipsoid.urdf.xacro (robot description, xacro)
@@ -37,22 +37,19 @@
     </link>
     <gazebo reference="${link_prefix}distal">
-      <sensor type="contact" name="${link_prefix}distal_contact_sensor">
-        <update_rate>100.0</update_rate>
+      <sensor type="contact" name="${link_prefix}distal_contact" >
+        <always_on>1</always_on>
+        <update_rate>1000.0</update_rate>
         <contact>
-          <collision>${link_prefix}distal_collision_geom</collision>
+          <collision>${link_prefix}distal_collision</collision>
+          <topic>${link_prefix}distal_collision</topic>
         </contact>
         <plugin name="${link_prefix}distal_gazebo_ros_bumper_controller" filename="libgazebo_ros_bumper.so">
-          <alwaysOn>true</alwaysOn>
-          <frameName>${link_prefix}distal</frameName>
           <updateRate>100.0</updateRate>
-          <bumperTopicName>${link_prefix}distal_bumper</bumperTopicName>
+	  <frameName>${link_prefix}distal</frameName>
+	  <bumperTopicName>contacts/${link_prefix}/distal</bumperTopicName>
         </plugin>
       </sensor>
-      <mu1 value="500.0" />
-      <mu2 value="500.0" />
-      <kp  value="10000000.0" />
-      <kd  value="1.0" />
-      <material>Gazebo/Grey</material>
       <selfCollide>true</selfCollide>
+      <material>LightGrey</material>
     </gazebo>
     <joint name="${joint_prefix}J1" type="revolute">

File: sr_description/hand/xacro/finger/knuckle/edc_muscle_knuckle.urdf.xacro (robot description, xacro)
@@ -31,14 +31,15 @@
     </link>
     <gazebo reference="${link_prefix}knuckle">
-      <sensor type="contact" name="${link_prefix}knuckle_contact_sensor">
-        <update_rate>100.0</update_rate>
+      <sensor type="contact" name="${link_prefix}knuckle_contact" >
+        <always_on>1</always_on>
+        <update_rate>1000.0</update_rate>
         <contact>
-          <collision>${link_prefix}knuckle_collision_geom</collision>
+          <collision>${link_prefix}knuckle_collision</collision>
+          <topic>${link_prefix}knuckle_collision</topic>
         </contact>
         <plugin name="${link_prefix}knuckle_gazebo_ros_bumper_controller" filename="libgazebo_ros_bumper.so">
-          <alwaysOn>true</alwaysOn>
-          <frameName>${link_prefix}knuckle</frameName>
           <updateRate>100.0</updateRate>
-          <bumperTopicName>${link_prefix}knuckle_bumper</bumperTopicName>
+	  <frameName>${link_prefix}knuckle</frameName>
+	  <bumperTopicName>contacts/${link_prefix}/knuckle</bumperTopicName>
         </plugin>
       </sensor>

File: sr_description/hand/xacro/finger/knuckle/knuckle.urdf.xacro (robot description, xacro)
@@ -31,14 +31,15 @@
     </link>
     <gazebo reference="${link_prefix}knuckle">
-      <sensor type="contact" name="${link_prefix}knuckle_contact_sensor">
-        <update_rate>100.0</update_rate>
+      <sensor type="contact" name="${link_prefix}knuckle_contact" >
+        <always_on>1</always_on>
+        <update_rate>1000.0</update_rate>
         <contact>
-          <collision>${link_prefix}knuckle_collision_geom</collision>
+          <collision>${link_prefix}knuckle_collision</collision>
+          <topic>${link_prefix}knuckle_collision</topic>
         </contact>
         <plugin name="${link_prefix}knuckle_gazebo_ros_bumper_controller" filename="libgazebo_ros_bumper.so">
-          <alwaysOn>true</alwaysOn>
-          <frameName>${link_prefix}knuckle</frameName>
           <updateRate>100.0</updateRate>
-          <bumperTopicName>${link_prefix}knuckle_bumper</bumperTopicName>
+	  <frameName>${link_prefix}knuckle</frameName>
+	  <bumperTopicName>contacts/${link_prefix}/knuckle</bumperTopicName>
         </plugin>
       </sensor>

File: sr_description/hand/xacro/finger/lfmetacarpal/edc_muscle_lfmetacarpal.urdf.xacro (robot description, xacro)
@@ -39,17 +39,18 @@
     </link>
     <gazebo reference="lfmetacarpal">
-      <sensor type="contact" name="lfmetacarpal_contact_sensor">
-        <update_rate>100.0</update_rate>
+      <sensor type="contact" name="lfmetacarpal_contact" >
+        <always_on>1</always_on>
+        <update_rate>1000.0</update_rate>
         <contact>
-          <collision>lfmetacarpal_collision_geom</collision>
+          <collision>lfmetacarpal_collision</collision>
+          <topic>lfmetacarpal_collision</topic>
         </contact>
         <plugin name="lfmetacarpal_gazebo_ros_bumper_controller" filename="libgazebo_ros_bumper.so">
-          <alwaysOn>true</alwaysOn>
-          <frameName>lfmetacarpal</frameName>
           <updateRate>100.0</updateRate>
-          <bumperTopicName>lfmetacarpal_bumper</bumperTopicName>
+	  <frameName>lfmetacarpal</frameName>
+	  <bumperTopicName>contacts/lf/metacarpal</bumperTopicName>
         </plugin>
       </sensor>
-      <material>Gazebo/Grey</material>
+      <material>LightGrey</material>
     </gazebo>
     <joint name="LFJ5" type="revolute">

File: sr_description/hand/xacro/finger/lfmetacarpal/lfmetacarpal.urdf.xacro (robot description, xacro)
@@ -39,17 +39,18 @@
     </link>
     <gazebo reference="lfmetacarpal">
-      <sensor type="contact" name="lfmetacarpal_contact_sensor">
-        <update_rate>100.0</update_rate>
+      <sensor type="contact" name="lfmetacarpal_contact" >
+        <always_on>1</always_on>
+        <update_rate>1000.0</update_rate>
         <contact>
-          <collision>lfmetacarpal_collision_geom</collision>
+          <collision>lfmetacarpal_collision</collision>
+          <topic>lfmetacarpal_collision</topic>
         </contact>
         <plugin name="lfmetacarpal_gazebo_ros_bumper_controller" filename="libgazebo_ros_bumper.so">
-          <alwaysOn>true</alwaysOn>
-          <frameName>lfmetacarpal</frameName>
           <updateRate>100.0</updateRate>
-          <bumperTopicName>lfmetacarpal_bumper</bumperTopicName>
+	  <frameName>lfmetacarpal</frameName>
+	  <bumperTopicName>contacts/lf/metacarpal</bumperTopicName>
         </plugin>
       </sensor>
-      <material>Gazebo/Grey</material>
+      <material>LightGrey</material>
     </gazebo>
     <joint name="LFJ5" type="revolute">

File: sr_description/hand/xacro/finger/little_finger_ellipsoid.urdf.xacro (robot description, xacro)
@@ -36,14 +36,15 @@
     </link>
     <gazebo reference="lfknuckle">
-      <sensor type="contact" name="lfknuckle_contact_sensor">
-        <update_rate>100.0</update_rate>
+      <sensor type="contact" name="lfknuckle_contact" >
+        <always_on>1</always_on>
+        <update_rate>1000.0</update_rate>
         <contact>
-          <collision>lfknuckle_collision_geom</collision>
+          <collision>lfknuckle_collision</collision>
+          <topic>lfknuckle_collision</topic>
         </contact>
         <plugin name="lfknuckle_gazebo_ros_bumper_controller" filename="libgazebo_ros_bumper.so">
-          <alwaysOn>true</alwaysOn>
-          <frameName>lfknuckle</frameName>
           <updateRate>100.0</updateRate>
-          <bumperTopicName>lfknuckle_bumper</bumperTopicName>
+	  <frameName>lfknuckle</frameName>
+	  <bumperTopicName>contacts/lf/knuckle</bumperTopicName>
         </plugin>
       </sensor>

File: sr_description/hand/xacro/finger/middle/middle.urdf.xacro (robot description, xacro)
@@ -30,18 +30,18 @@
     </link>
     <gazebo reference="${link_prefix}middle">
-      <sensor type="contact" name="${link_prefix}middle_contact_sensor">
-        <update_rate>100.0</update_rate>
+      <sensor type="contact" name="${link_prefix}middle_contact" >
+        <always_on>1</always_on>
+        <update_rate>1000.0</update_rate>
         <contact>
-          <collision>${link_prefix}middle_collision_geom</collision>
+          <collision>${link_prefix}middle_collision</collision>
+          <topic>${link_prefix}middle_collision</topic>
         </contact>
         <plugin name="${link_prefix}middle_gazebo_ros_bumper_controller" filename="libgazebo_ros_bumper.so">
-          <alwaysOn>true</alwaysOn>
-          <frameName>${link_prefix}middle</frameName>
           <updateRate>100.0</updateRate>
-          <bumperTopicName>${link_prefix}middle_bumper</bumperTopicName>
+	  <frameName>${link_prefix}middle</frameName>
+	  <bumperTopicName>contacts/${link_prefix}/middle</bumperTopicName>
         </plugin>
       </sensor>
-      <material>Gazebo/Grey</material>
-      <selfCollide>true</selfCollide>
+      <material>LightGrey</material>
     </gazebo>
     <joint name="${joint_prefix}J2" type="revolute">

File: sr_description/hand/xacro/finger/proximal/edc_muscle_proximal.urdf.xacro (robot description, xacro)
@@ -30,18 +30,18 @@
     </link>
     <gazebo reference="${link_prefix}proximal">
-      <sensor type="contact" name="${link_prefix}proximal_contact_sensor">
-        <update_rate>100.0</update_rate>
+      <sensor type="contact" name="${link_prefix}proximal_contact" >
+        <always_on>1</always_on>
+        <update_rate>1000.0</update_rate>
         <contact>
-          <collision>${link_prefix}proximal_collision_geom</collision>
+          <collision>${link_prefix}proximal_collision</collision>
+          <topic>${link_prefix}proximal_collision</topic>
         </contact>
         <plugin name="${link_prefix}proximal_gazebo_ros_bumper_controller" filename="libgazebo_ros_bumper.so">
-          <alwaysOn>true</alwaysOn>
-          <frameName>${link_prefix}proximal</frameName>
           <updateRate>100.0</updateRate>
-          <bumperTopicName>${link_prefix}proximal_bumper</bumperTopicName>
+	  <frameName>${link_prefix}proximal</frameName>
+	  <bumperTopicName>contacts/${link_prefix}/proximal</bumperTopicName>
         </plugin>
       </sensor>
-      <material>Gazebo/Grey</material>
-      <selfCollide>true</selfCollide>
+      <material>LightGrey</material>
     </gazebo>
     <joint name="${joint_prefix}J3" type="revolute">

File: sr_description/hand/xacro/finger/proximal/proximal.urdf.xacro (robot description, xacro)
@@ -30,18 +30,18 @@
     </link>
     <gazebo reference="${link_prefix}proximal">
-      <sensor type="contact" name="${link_prefix}proximal_contact_sensor">
-        <update_rate>100.0</update_rate>
+      <sensor type="contact" name="${link_prefix}proximal_contact" >
+        <always_on>1</always_on>
+        <update_rate>1000.0</update_rate>
         <contact>
-          <collision>${link_prefix}proximal_collision_geom</collision>
+          <collision>${link_prefix}proximal_collision</collision>
+          <topic>${link_prefix}proximal_collision</topic>
         </contact>
         <plugin name="${link_prefix}proximal_gazebo_ros_bumper_controller" filename="libgazebo_ros_bumper.so">
-          <alwaysOn>true</alwaysOn>
-          <frameName>${link_prefix}proximal</frameName>
           <updateRate>100.0</updateRate>
-          <bumperTopicName>${link_prefix}proximal_bumper</bumperTopicName>
+	  <frameName>${link_prefix}proximal</frameName>
+	  <bumperTopicName>contacts/${link_prefix}/proximal</bumperTopicName>
         </plugin>
       </sensor>
-      <material>Gazebo/Grey</material>
-      <selfCollide>true</selfCollide>
+      <material>LightGrey</material>
     </gazebo>
     <joint name="${joint_prefix}J3" type="revolute">

File: sr_description/hand/xacro/forearm/forearm_motor.urdf.xacro (robot description, xacro)
@@ -23,5 +23,5 @@
     </link>
     <gazebo reference="forearm">
-      <material>Gazebo/Grey</material>
+      <material>LightGrey</material>
       <selfCollide>false</selfCollide>
     </gazebo>

File: sr_description/hand/xacro/forearm/forearm_muscle.urdf.xacro (robot description, xacro)
@@ -23,5 +23,5 @@
     </link>
     <gazebo reference="forearm">
-      <material>Gazebo/Grey</material>
+      <material>LightGrey</material>
       <selfCollide>false</selfCollide>
     </gazebo>

File: sr_description/hand/xacro/palm/edc_muscle_palm.urdf.xacro (robot description, xacro)
@@ -39,17 +39,18 @@
     </link>
     <gazebo reference="palm">
-      <sensor type="contact" name="palm_contact_sensor">
-        <update_rate>100.0</update_rate>
+      <sensor type="contact" name="palm_contact" >
+        <always_on>1</always_on>
+        <update_rate>1000.0</update_rate>
         <contact>
-          <collision>palm_collision_geom</collision>
+          <collision>palm_collision</collision>
+          <topic>palm_collision</topic>
         </contact>
         <plugin name="palm_gazebo_ros_bumper_controller" filename="libgazebo_ros_bumper.so">
-          <alwaysOn>true</alwaysOn>
-          <frameName>palm</frameName>
           <updateRate>100.0</updateRate>
-          <bumperTopicName>palm_bumper</bumperTopicName>
+	  <frameName>palm</frameName>
+	  <bumperTopicName>contacts/palm</bumperTopicName>
         </plugin>
       </sensor>
-      <material>Gazebo/Grey</material>
+      <material>LightGrey</material>
     </gazebo>
     <joint name="WRJ1" type="revolute">

File: sr_description/hand/xacro/palm/palm.urdf.xacro (robot description, xacro)
@@ -39,17 +39,18 @@
     </link>
     <gazebo reference="palm">
-      <sensor type="contact" name="palm_contact_sensor">
-        <update_rate>100.0</update_rate>
+      <sensor type="contact" name="palm_contact" >
+        <always_on>1</always_on>
+        <update_rate>1000.0</update_rate>
         <contact>
-          <collision>palm_collision_geom</collision>
+          <collision>palm_collision</collision>
+          <topic>palm_collision</topic>
         </contact>
         <plugin name="palm_gazebo_ros_bumper_controller" filename="libgazebo_ros_bumper.so">
-          <alwaysOn>true</alwaysOn>
-          <frameName>palm</frameName>
           <updateRate>100.0</updateRate>
-          <bumperTopicName>palm_bumper</bumperTopicName>
+	  <frameName>palm</frameName>
+	  <bumperTopicName>contacts/palm</bumperTopicName>
         </plugin>
       </sensor>
-      <material>Gazebo/Grey</material>
+      <material>LightGrey</material>
     </gazebo>
     <joint name="WRJ1" type="revolute">
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