Commit message: Imported upstream version '1.3.1' of 'upstream'

File: sr_description/arm/xacro/hand_support/shadowarm_handsupport_motor.transmission.xacro (robot description, xacro)
@@ -8,7 +8,4 @@
       <actuator name="forearm_rotation" />
       <joint name="ElbowJRotate" />
-      <mechanicalReduction>1</mechanicalReduction>
-      <motorTorqueConstant>1</motorTorqueConstant>
-      <pulsesPerRevolution>90000</pulsesPerRevolution>
     </transmission>
   </xacro:macro>

File: sr_description/arm/xacro/hand_support/shadowarm_handsupport_muscle.transmission.xacro (robot description, xacro)
@@ -8,7 +8,4 @@
       <actuator name="forearm_rotation" />
       <joint name="ElbowJRotate" />
-      <mechanicalReduction>1</mechanicalReduction>
-      <motorTorqueConstant>1</motorTorqueConstant>
-      <pulsesPerRevolution>90000</pulsesPerRevolution>
     </transmission>
   </xacro:macro>

File: sr_description/arm/xacro/lower_arm/shadowarm_lowerarm.transmission.xacro (robot description, xacro)
@@ -8,7 +8,4 @@
       <actuator name="elbow_abduction" />
       <joint name="ElbowJSwing" />
-      <mechanicalReduction>1</mechanicalReduction>
-      <motorTorqueConstant>1</motorTorqueConstant>
-      <pulsesPerRevolution>90000</pulsesPerRevolution>
     </transmission>
   </xacro:macro>

File: sr_description/arm/xacro/trunk/shadowarm_trunk.transmission.xacro (robot description, xacro)
@@ -8,7 +8,4 @@
       <actuator name="trunk_rotation" />
       <joint name="ShoulderJRotate" />
-      <mechanicalReduction>1</mechanicalReduction>
-      <motorTorqueConstant>1</motorTorqueConstant>
-      <pulsesPerRevolution>90000</pulsesPerRevolution>
     </transmission>
   </xacro:macro>

File: sr_description/arm/xacro/upper_arm/shadowarm_upperarm.transmission.xacro (robot description, xacro)
@@ -8,7 +8,4 @@
       <actuator name="shoulder_rotation" />
       <joint name="ShoulderJSwing" />
-      <mechanicalReduction>1</mechanicalReduction>
-      <motorTorqueConstant>1</motorTorqueConstant>
-      <pulsesPerRevolution>90000</pulsesPerRevolution>
     </transmission>
   </xacro:macro>

File: sr_description/hand/xacro/finger/biotac/biotac.transmission.xacro (robot description, xacro)
@@ -11,9 +11,6 @@
     <transmission type="sr_mechanism_model/J0Transmission" name="${link_prefix}middle_transmission">
       <actuator name="${joint_prefix}J0" />
-      <joint1 name="${joint_prefix}J1" />
-      <joint2 name="${joint_prefix}J2" />
-      <mechanicalReduction>1</mechanicalReduction>
-      <motorTorqueConstant>1</motorTorqueConstant>
-      <pulsesPerRevolution>90000</pulsesPerRevolution>
+      <joint name="${joint_prefix}J1" />
+      <joint name="${joint_prefix}J2" />
     </transmission>
   </xacro:macro>

File: sr_description/hand/xacro/finger/biotac/edc_muscle_biotac.transmission.xacro (robot description, xacro)
@@ -11,9 +11,6 @@
     <transmission type="sr_mechanism_model/J0TransmissionForMuscle" name="${link_prefix}middle_transmission">
       <actuator name="${joint_prefix}J0" />
-      <joint1 name="${joint_prefix}J1" />
-      <joint2 name="${joint_prefix}J2" />
-      <mechanicalReduction>1</mechanicalReduction>
-      <motorTorqueConstant>1</motorTorqueConstant>
-      <pulsesPerRevolution>90000</pulsesPerRevolution>
+      <joint name="${joint_prefix}J1" />
+      <joint name="${joint_prefix}J2" />
     </transmission>
   </xacro:macro>

File: sr_description/hand/xacro/finger/distal/distal.transmission.xacro (robot description, xacro)
@@ -8,7 +8,4 @@
       <actuator name="${joint_prefix}J1" />
       <joint name="${joint_prefix}J1" />
-      <mechanicalReduction>1</mechanicalReduction>
-      <motorTorqueConstant>1</motorTorqueConstant>
-      <pulsesPerRevolution>90000</pulsesPerRevolution>
     </transmission>
   </xacro:macro>

File: sr_description/hand/xacro/finger/distal/distal_ellipsoid.urdf.xacro (robot description, xacro)
@@ -7,5 +7,5 @@
        xmlns:geom="http://playerstage.sourceforge.net/gazebo/xmlschema/#geom">
   <xacro:include filename="$(find sr_description)/hand/xacro/finger/distal/distal.transmission.xacro" />
-  <xacro:macro name="distal" params="link_prefix joint_prefix parent">
+  <xacro:macro name="distal_ellipsoid" params="link_prefix joint_prefix parent">
     <link name="${link_prefix}distal">
       <inertial>

File: sr_description/hand/xacro/finger/knuckle/edc_muscle_knuckle.transmission.xacro (robot description, xacro)
@@ -8,7 +8,4 @@
       <actuator name="${joint_prefix}J4" />
       <joint name="${joint_prefix}J4" />
-      <mechanicalReduction>1</mechanicalReduction>
-      <motorTorqueConstant>1</motorTorqueConstant>
-      <pulsesPerRevolution>90000</pulsesPerRevolution>
     </transmission>
   </xacro:macro>

File: sr_description/hand/xacro/finger/knuckle/knuckle.transmission.xacro (robot description, xacro)
@@ -8,7 +8,4 @@
       <actuator name="${joint_prefix}J4" />
       <joint name="${joint_prefix}J4" />
-      <mechanicalReduction>1</mechanicalReduction>
-      <motorTorqueConstant>1</motorTorqueConstant>
-      <pulsesPerRevolution>90000</pulsesPerRevolution>
     </transmission>
   </xacro:macro>

File: sr_description/hand/xacro/finger/lfmetacarpal/edc_muscle_lfmetacarpal.transmission.xacro (robot description, xacro)
@@ -8,7 +8,4 @@
       <actuator name="LFJ5" />
       <joint name="LFJ5" />
-      <mechanicalReduction>1</mechanicalReduction>
-      <motorTorqueConstant>1</motorTorqueConstant>
-      <pulsesPerRevolution>90000</pulsesPerRevolution>
     </transmission>
   </xacro:macro>

File: sr_description/hand/xacro/finger/lfmetacarpal/lfmetacarpal.transmission.xacro (robot description, xacro)
@@ -8,7 +8,4 @@
       <actuator name="LFJ5" />
       <joint name="LFJ5" />
-      <mechanicalReduction>1</mechanicalReduction>
-      <motorTorqueConstant>1</motorTorqueConstant>
-      <pulsesPerRevolution>90000</pulsesPerRevolution>
     </transmission>
   </xacro:macro>

File: sr_description/hand/xacro/finger/little_finger_ellipsoid.urdf.xacro (robot description, xacro)
@@ -11,5 +11,5 @@
   <xacro:include filename="$(find sr_description)/hand/xacro/finger/distal/distal_ellipsoid.urdf.xacro" />
   <xacro:include filename="$(find sr_description)/hand/xacro/finger/lfmetacarpal/lfmetacarpal.urdf.xacro" />
-  <xacro:macro name="little_finger" params="link_prefix joint_prefix parent">
+  <xacro:macro name="little_finger_ellipsoid" params="link_prefix joint_prefix parent">
     <xacro:lfmetacarpal parent="${parent}" >
     </xacro:lfmetacarpal>
@@ -63,7 +63,4 @@
       <actuator name="LFJ4" />
       <joint name="LFJ4" />
-      <mechanicalReduction>1</mechanicalReduction>
-      <motorTorqueConstant>1</motorTorqueConstant>
-      <pulsesPerRevolution>90000</pulsesPerRevolution>
     </transmission>
     <xacro:proximal link_prefix="${link_prefix}" joint_prefix="${joint_prefix}" parent="${link_prefix}knuckle" >

File: sr_description/hand/xacro/finger/middle/middle.transmission.xacro (robot description, xacro)
@@ -7,9 +7,6 @@
     <transmission type="sr_mechanism_model/J0Transmission" name="${link_prefix}middle_transmission">
       <actuator name="${joint_prefix}J0" />
-      <joint1 name="${joint_prefix}J1" />
-      <joint2 name="${joint_prefix}J2" />
-      <mechanicalReduction>1</mechanicalReduction>
-      <motorTorqueConstant>1</motorTorqueConstant>
-      <pulsesPerRevolution>90000</pulsesPerRevolution>
+      <joint name="${joint_prefix}J1" />
+      <joint name="${joint_prefix}J2" />
     </transmission>
   </xacro:macro>

File: sr_description/hand/xacro/finger/proximal/edc_muscle_proximal.transmission.xacro (robot description, xacro)
@@ -8,7 +8,4 @@
       <actuator name="${joint_prefix}J3" />
       <joint name="${joint_prefix}J3" />
-      <mechanicalReduction>1</mechanicalReduction>
-      <motorTorqueConstant>1</motorTorqueConstant>
-      <pulsesPerRevolution>90000</pulsesPerRevolution>
     </transmission>
   </xacro:macro>

File: sr_description/hand/xacro/finger/proximal/proximal.transmission.xacro (robot description, xacro)
@@ -8,7 +8,4 @@
       <actuator name="${joint_prefix}J3" />
       <joint name="${joint_prefix}J3" />
-      <mechanicalReduction>1</mechanicalReduction>
-      <motorTorqueConstant>1</motorTorqueConstant>
-      <pulsesPerRevolution>90000</pulsesPerRevolution>
     </transmission>
   </xacro:macro>

File: sr_description/hand/xacro/full_hand_motor_ellipsoid.urdf.xacro (robot description, xacro)
@@ -17,20 +17,20 @@
     <xacro:palm parent="wrist">
     </xacro:palm>
-    <xacro:finger link_prefix="ff" joint_prefix="FF" parent="palm">
+    <xacro:finger_ellipsoid link_prefix="ff" joint_prefix="FF" parent="palm">
       <origin xyz="0.033 0 0.095" rpy="0 0 0" />
       <axis xyz="0 -1 0" />
-    </xacro:finger>
-    <xacro:finger link_prefix="mf" joint_prefix="MF" parent="palm">
+    </xacro:finger_ellipsoid>
+    <xacro:finger_ellipsoid link_prefix="mf" joint_prefix="MF" parent="palm">
       <origin xyz="0.011 0 0.099" rpy="0 0 0" />
       <axis xyz="0 -1 0" />
-    </xacro:finger>
-    <xacro:finger link_prefix="rf" joint_prefix="RF" parent="palm">
+    </xacro:finger_ellipsoid>
+    <xacro:finger_ellipsoid link_prefix="rf" joint_prefix="RF" parent="palm">
       <origin xyz="-0.011 0 0.095" rpy="0 0 0" />
       <axis xyz="0 1 0" />
-    </xacro:finger>
-    <xacro:little_finger link_prefix="lf" joint_prefix="LF" parent="palm">
-    </xacro:little_finger>
-    <xacro:thumb parent="palm">
-    </xacro:thumb>
+    </xacro:finger_ellipsoid>
+    <xacro:little_finger_ellipsoid link_prefix="lf" joint_prefix="LF" parent="palm">
+    </xacro:little_finger_ellipsoid>
+    <xacro:thumb_ellipsoid parent="palm">
+    </xacro:thumb_ellipsoid>
   </xacro:macro>
 </robot>

File: sr_description/hand/xacro/palm/edc_muscle_palm.transmission.xacro (robot description, xacro)
@@ -8,7 +8,4 @@
       <actuator name="WRJ1" />
       <joint name="WRJ1" />
-      <mechanicalReduction>1</mechanicalReduction>
-      <motorTorqueConstant>1</motorTorqueConstant>
-      <pulsesPerRevolution>90000</pulsesPerRevolution>
     </transmission>
   </xacro:macro>

File: sr_description/hand/xacro/palm/palm.transmission.xacro (robot description, xacro)
@@ -8,7 +8,4 @@
       <actuator name="WRJ1" />
       <joint name="WRJ1" />
-      <mechanicalReduction>1</mechanicalReduction>
-      <motorTorqueConstant>1</motorTorqueConstant>
-      <pulsesPerRevolution>90000</pulsesPerRevolution>
     </transmission>
   </xacro:macro>
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