Commit message: Imported upstream version '1.3.4' of 'upstream'

File: sr_description/arm/xacro/hand_support/shadowarm_handsupport_motor.transmission.xacro (robot description, xacro)
@@ -8,4 +8,7 @@
       <actuator name="forearm_rotation" />
       <joint name="ElbowJRotate" />
+      <mechanicalReduction>1</mechanicalReduction>
+      <motorTorqueConstant>1</motorTorqueConstant>
+      <pulsesPerRevolution>90000</pulsesPerRevolution>
     </transmission>
   </xacro:macro>

File: sr_description/arm/xacro/hand_support/shadowarm_handsupport_muscle.transmission.xacro (robot description, xacro)
@@ -8,4 +8,7 @@
       <actuator name="forearm_rotation" />
       <joint name="ElbowJRotate" />
+      <mechanicalReduction>1</mechanicalReduction>
+      <motorTorqueConstant>1</motorTorqueConstant>
+      <pulsesPerRevolution>90000</pulsesPerRevolution>
     </transmission>
   </xacro:macro>

File: sr_description/arm/xacro/lower_arm/shadowarm_lowerarm.transmission.xacro (robot description, xacro)
@@ -8,4 +8,7 @@
       <actuator name="elbow_abduction" />
       <joint name="ElbowJSwing" />
+      <mechanicalReduction>1</mechanicalReduction>
+      <motorTorqueConstant>1</motorTorqueConstant>
+      <pulsesPerRevolution>90000</pulsesPerRevolution>
     </transmission>
   </xacro:macro>

File: sr_description/arm/xacro/trunk/shadowarm_trunk.transmission.xacro (robot description, xacro)
@@ -8,4 +8,7 @@
       <actuator name="trunk_rotation" />
       <joint name="ShoulderJRotate" />
+      <mechanicalReduction>1</mechanicalReduction>
+      <motorTorqueConstant>1</motorTorqueConstant>
+      <pulsesPerRevolution>90000</pulsesPerRevolution>
     </transmission>
   </xacro:macro>

File: sr_description/arm/xacro/upper_arm/shadowarm_upperarm.transmission.xacro (robot description, xacro)
@@ -8,4 +8,7 @@
       <actuator name="shoulder_rotation" />
       <joint name="ShoulderJSwing" />
+      <mechanicalReduction>1</mechanicalReduction>
+      <motorTorqueConstant>1</motorTorqueConstant>
+      <pulsesPerRevolution>90000</pulsesPerRevolution>
     </transmission>
   </xacro:macro>

File: sr_description/hand/xacro/finger/biotac/biotac.transmission.xacro (robot description, xacro)
@@ -11,6 +11,9 @@
     <transmission type="sr_mechanism_model/J0Transmission" name="${link_prefix}middle_transmission">
       <actuator name="${joint_prefix}J0" />
-      <joint name="${joint_prefix}J1" />
-      <joint name="${joint_prefix}J2" />
+      <joint1 name="${joint_prefix}J1" />
+      <joint2 name="${joint_prefix}J2" />
+      <mechanicalReduction>1</mechanicalReduction>
+      <motorTorqueConstant>1</motorTorqueConstant>
+      <pulsesPerRevolution>90000</pulsesPerRevolution>
     </transmission>
   </xacro:macro>

File: sr_description/hand/xacro/finger/biotac/edc_muscle_biotac.transmission.xacro (robot description, xacro)
@@ -11,6 +11,9 @@
     <transmission type="sr_mechanism_model/J0TransmissionForMuscle" name="${link_prefix}middle_transmission">
       <actuator name="${joint_prefix}J0" />
-      <joint name="${joint_prefix}J1" />
-      <joint name="${joint_prefix}J2" />
+      <joint1 name="${joint_prefix}J1" />
+      <joint2 name="${joint_prefix}J2" />
+      <mechanicalReduction>1</mechanicalReduction>
+      <motorTorqueConstant>1</motorTorqueConstant>
+      <pulsesPerRevolution>90000</pulsesPerRevolution>
     </transmission>
   </xacro:macro>

File: sr_description/hand/xacro/finger/distal/distal.transmission.xacro (robot description, xacro)
@@ -8,4 +8,7 @@
       <actuator name="${joint_prefix}J1" />
       <joint name="${joint_prefix}J1" />
+      <mechanicalReduction>1</mechanicalReduction>
+      <motorTorqueConstant>1</motorTorqueConstant>
+      <pulsesPerRevolution>90000</pulsesPerRevolution>
     </transmission>
   </xacro:macro>

File: sr_description/hand/xacro/finger/distal/distal_ellipsoid.urdf.xacro (robot description, xacro)
@@ -12,6 +12,6 @@
 	<mass value="0.010" />
 	<origin xyz="0 0 0.013" />
-	<inertia  ixx="0.1" ixy="0.0"  ixz="0.0"  iyy="0.1"  iyz="0.0"
-		  izz="0.0" />
+	<inertia ixx="0.001" ixy="0.0" ixz="0.0" iyy="0.001" iyz="0.0"
+	izz="0.00025" />
       </inertial>
       <visual>
@@ -58,7 +58,6 @@
       <origin xyz="0 0 0.025" rpy="0 0 0" />
       <axis xyz="1 0 0" />
-      <limit lower="0" upper="${M_PI/2}" effort="1000.0"
-	     velocity="10.0" />
-      <dynamics damping="10.0"/>
+      <limit lower="0" upper="${M_PI/2}" effort="2" velocity="1.0" />
+      <dynamics damping="0.1"/>
     </joint>
     <link name="${link_prefix}tip">

File: sr_description/hand/xacro/finger/knuckle/edc_muscle_knuckle.transmission.xacro (robot description, xacro)
@@ -8,4 +8,7 @@
       <actuator name="${joint_prefix}J4" />
       <joint name="${joint_prefix}J4" />
+      <mechanicalReduction>1</mechanicalReduction>
+      <motorTorqueConstant>1</motorTorqueConstant>
+      <pulsesPerRevolution>90000</pulsesPerRevolution>
     </transmission>
   </xacro:macro>

File: sr_description/hand/xacro/finger/knuckle/knuckle.transmission.xacro (robot description, xacro)
@@ -8,4 +8,7 @@
       <actuator name="${joint_prefix}J4" />
       <joint name="${joint_prefix}J4" />
+      <mechanicalReduction>1</mechanicalReduction>
+      <motorTorqueConstant>1</motorTorqueConstant>
+      <pulsesPerRevolution>90000</pulsesPerRevolution>
     </transmission>
   </xacro:macro>

File: sr_description/hand/xacro/finger/lfmetacarpal/edc_muscle_lfmetacarpal.transmission.xacro (robot description, xacro)
@@ -8,4 +8,7 @@
       <actuator name="LFJ5" />
       <joint name="LFJ5" />
+      <mechanicalReduction>1</mechanicalReduction>
+      <motorTorqueConstant>1</motorTorqueConstant>
+      <pulsesPerRevolution>90000</pulsesPerRevolution>
     </transmission>
   </xacro:macro>

File: sr_description/hand/xacro/finger/lfmetacarpal/lfmetacarpal.transmission.xacro (robot description, xacro)
@@ -8,4 +8,7 @@
       <actuator name="LFJ5" />
       <joint name="LFJ5" />
+      <mechanicalReduction>1</mechanicalReduction>
+      <motorTorqueConstant>1</motorTorqueConstant>
+      <pulsesPerRevolution>90000</pulsesPerRevolution>
     </transmission>
   </xacro:macro>

File: sr_description/hand/xacro/finger/little_finger_ellipsoid.urdf.xacro (robot description, xacro)
@@ -6,68 +6,21 @@
        xmlns:body="http://playerstage.sourceforge.net/gazebo/xmlschema/#body"
        xmlns:geom="http://playerstage.sourceforge.net/gazebo/xmlschema/#geom">
-  <xacro:include filename="$(find sr_description)/hand/xacro/finger/knuckle/knuckle.urdf.xacro" />
-  <xacro:include filename="$(find sr_description)/hand/xacro/finger/proximal/proximal.urdf.xacro" />
-  <xacro:include filename="$(find sr_description)/hand/xacro/finger/middle/middle.urdf.xacro" />
-  <xacro:include filename="$(find sr_description)/hand/xacro/finger/distal/distal_ellipsoid.urdf.xacro" />
   <xacro:include filename="$(find sr_description)/hand/xacro/finger/lfmetacarpal/lfmetacarpal.urdf.xacro" />
-  <xacro:macro name="little_finger_ellipsoid" params="link_prefix joint_prefix parent">
-    <xacro:lfmetacarpal parent="${parent}" >
-    </xacro:lfmetacarpal>
-    <link name="lfknuckle">
-      <inertial>
-	<origin xyz="0 0 0.06579" rpy="0 0 0" />
-	<mass value="0.008" />
-	<inertia  ixx="0.1" ixy="0.0"  ixz="0.0"  iyy="0.1"  iyz="0.0"
-	izz="0.1" />
-      </inertial>
-      <visual>
-	<origin xyz="0 0 0" rpy="0 0 0" />
-	<geometry name="knuckle_visual">
-      <mesh filename="package://sr_description/hand/model/knuckle.dae" scale="0.001 0.001 0.001" />
-      </geometry>
-      <material name="LightGrey" />
-      </visual>
-      <collision>
-	<origin xyz="0 0 0" rpy="0 0 0" />
-	<geometry name="knuckle_collision_geom">
-	  <box size="0.005 0.005 0.005" />
-	</geometry>
-      </collision>
-    </link>
-    <gazebo reference="lfknuckle">
-      <sensor type="contact" name="lfknuckle_contact" >
-        <always_on>1</always_on>
-        <update_rate>1000.0</update_rate>
-        <contact>
-          <collision>lfknuckle_collision</collision>
-          <topic>lfknuckle_collision</topic>
-        </contact>
-        <plugin name="lfknuckle_gazebo_ros_bumper_controller" filename="libgazebo_ros_bumper.so">
-          <updateRate>100.0</updateRate>
-	  <frameName>lfknuckle</frameName>
-	  <bumperTopicName>contacts/lf/knuckle</bumperTopicName>
-        </plugin>
-      </sensor>
-      <material>Gazebo/Grey</material>
-    </gazebo>
-    <joint name="LFJ4" type="revolute">
-      <parent link="lfmetacarpal"/>
-      <child link="lfknuckle"/>
+  <xacro:include filename="$(find sr_description)/hand/xacro/finger/classic_finger_ellipsoid.urdf.xacro" />
+  <!-- Right Handed -->
+  <xacro:macro name="little_finger" params="link_prefix joint_prefix parent">
+    <xacro:lfmetacarpal parent="${parent}" />
+    <xacro:finger_ellipsoid link_prefix="${link_prefix}" joint_prefix="${joint_prefix}" parent="lfmetacarpal">
       <origin xyz="0 0 0.06579" rpy="0 0 0" />
       <axis xyz="0 1 0" />
-      <limit lower="-0.3491" upper="0.3491"
-      effort="1000.0" velocity="10.0"/>
-      <dynamics damping="10.0"/>
-    </joint>
-    <transmission type="sr_mechanism_model/SimpleTransmission" name="lfknuckle_transmission">
-      <actuator name="LFJ4" />
-      <joint name="LFJ4" />
-    </transmission>
-    <xacro:proximal link_prefix="${link_prefix}" joint_prefix="${joint_prefix}" parent="${link_prefix}knuckle" >
-    </xacro:proximal>
-    <xacro:middle link_prefix="${link_prefix}" joint_prefix="${joint_prefix}" parent="${link_prefix}proximal" >
-    </xacro:middle>
-    <xacro:distal link_prefix="${link_prefix}" joint_prefix="${joint_prefix}" parent="${link_prefix}middle" >
-    </xacro:distal>
+    </xacro:finger_ellipsoid>
+  </xacro:macro>
+  <!-- Left Handed -->
+  <xacro:macro name="little_finger_left" params="link_prefix joint_prefix parent">
+    <xacro:lfmetacarpal_left parent="${parent}" />
+    <xacro:finger_ellipsoid link_prefix="${link_prefix}" joint_prefix="${joint_prefix}" parent="lfmetacarpal">
+      <origin xyz="0 0 0.06579" rpy="0 0 0" />
+      <axis xyz="0 -1 0" />
+    </xacro:finger_ellipsoid>
   </xacro:macro>
 </robot>

File: sr_description/hand/xacro/finger/middle/middle.transmission.xacro (robot description, xacro)
@@ -7,6 +7,9 @@
     <transmission type="sr_mechanism_model/J0Transmission" name="${link_prefix}middle_transmission">
       <actuator name="${joint_prefix}J0" />
-      <joint name="${joint_prefix}J1" />
-      <joint name="${joint_prefix}J2" />
+      <joint1 name="${joint_prefix}J1" />
+      <joint2 name="${joint_prefix}J2" />
+      <mechanicalReduction>1</mechanicalReduction>
+      <motorTorqueConstant>1</motorTorqueConstant>
+      <pulsesPerRevolution>90000</pulsesPerRevolution>
     </transmission>
   </xacro:macro>

File: sr_description/hand/xacro/finger/proximal/edc_muscle_proximal.transmission.xacro (robot description, xacro)
@@ -8,4 +8,7 @@
       <actuator name="${joint_prefix}J3" />
       <joint name="${joint_prefix}J3" />
+      <mechanicalReduction>1</mechanicalReduction>
+      <motorTorqueConstant>1</motorTorqueConstant>
+      <pulsesPerRevolution>90000</pulsesPerRevolution>
     </transmission>
   </xacro:macro>

File: sr_description/hand/xacro/finger/proximal/proximal.transmission.xacro (robot description, xacro)
@@ -8,4 +8,7 @@
       <actuator name="${joint_prefix}J3" />
       <joint name="${joint_prefix}J3" />
+      <mechanicalReduction>1</mechanicalReduction>
+      <motorTorqueConstant>1</motorTorqueConstant>
+      <pulsesPerRevolution>90000</pulsesPerRevolution>
     </transmission>
   </xacro:macro>

File: sr_description/hand/xacro/full_hand_motor_ellipsoid.urdf.xacro (robot description, xacro)
@@ -29,6 +29,6 @@
       <axis xyz="0 1 0" />
     </xacro:finger_ellipsoid>
-    <xacro:little_finger_ellipsoid link_prefix="lf" joint_prefix="LF" parent="palm">
-    </xacro:little_finger_ellipsoid>
+    <xacro:little_finger link_prefix="lf" joint_prefix="LF" parent="palm">
+    </xacro:little_finger>
     <xacro:thumb_ellipsoid parent="palm">
     </xacro:thumb_ellipsoid>

File: sr_description/hand/xacro/palm/edc_muscle_palm.transmission.xacro (robot description, xacro)
@@ -8,4 +8,7 @@
       <actuator name="WRJ1" />
       <joint name="WRJ1" />
+      <mechanicalReduction>1</mechanicalReduction>
+      <motorTorqueConstant>1</motorTorqueConstant>
+      <pulsesPerRevolution>90000</pulsesPerRevolution>
     </transmission>
   </xacro:macro>

File: sr_description/hand/xacro/palm/palm.transmission.xacro (robot description, xacro)
@@ -8,4 +8,7 @@
       <actuator name="WRJ1" />
       <joint name="WRJ1" />
+      <mechanicalReduction>1</mechanicalReduction>
+      <motorTorqueConstant>1</motorTorqueConstant>
+      <pulsesPerRevolution>90000</pulsesPerRevolution>
     </transmission>
   </xacro:macro>
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