Commit message: Rebase from 'upstream'

File: sr_description/arm/xacro/base/shadowarm_base.urdf.xacro (robot description, xacro)
@@ -2,29 +2,28 @@
 <property name="M_PI" value="3.1415926535897931" />
 <xacro:macro name="shadowarm_base">
-    <link name="shadowarm_base">
-      <inertial>
-	<origin xyz="0 0 0.0" rpy="0 0 0" />
-	<mass value="0.4" />
-	<inertia  ixx="0.1" ixy="0.0"  ixz="0.0"  iyy="0.1"  iyz="0.0"
-	izz="0.0" />
-      </inertial>
-      <visual>
-	<origin xyz="0 0 0" rpy="0 0 0" />
-	<geometry name="shadowarm_visual">
-          <mesh filename="package://sr_description/arm/model/arm_base.dae" scale="0.001 0.001 0.001" />
-        </geometry>
-        <material name="Grey" />
-      </visual>
-      <collision>
-	<origin xyz="0 0 0.0" rpy="0 0 0" />
-	<geometry name="shadowarm_collision_geom">
-          <mesh filename="package://sr_description/arm/model/arm_base.dae" scale="0.001 0.001 0.001" />
-	</geometry>
-      </collision>
-    </link>
-    <gazebo reference="shadowarm_base">
-      <material>Gazebo/Grey</material>
-      <selfCollide>false</selfCollide>
-    </gazebo>
+  <link name="shadowarm_base">
+    <inertial>
+      <origin xyz="0 0 0" rpy="0 0 0"/>
+      <mass value="0.4" />
+      <inertia  ixx="0.1" ixy="0.0"  ixz="0.0"  iyy="0.1"  iyz="0.0"  izz="0.1" />
+    </inertial>
+    <visual>
+      <origin xyz="0 0 0" rpy="0 0 0"/>
+      <geometry name="shadowarm_base_visual">
+        <mesh filename="package://sr_description/arm/model/arm_base.dae" scale="0.001 0.001 0.001" />
+      </geometry>
+      <material name="LightGrey" />
+    </visual>
+    <collision>
+      <origin xyz="0 0 0.005" rpy="0 0 0" />
+      <geometry name="shadowarm_base_collision">
+        <box size="0.145 0.145 0.012"/>
+      </geometry>
+    </collision>
+  </link>
+  <gazebo reference="shadowarm_base">
+    <material>LightGrey</material>
+    <selfCollide>false</selfCollide>
+  </gazebo>
 </xacro:macro>
 </robot>

File: sr_description/arm/xacro/hand_support/shadowarm_handsupport_motor.urdf.xacro (robot description, xacro)
@@ -6,5 +6,5 @@
 	<origin xyz="0 0 0" rpy="0 0 0" />
 	<mass value="0.75" />
-	<inertia  ixx="1.0" ixy="0.0"  ixz="0.0"  iyy="0.0"  iyz="0.0"  izz="0.0" />
+	<inertia  ixx="0.01" ixy="0.0"  ixz="0.0"  iyy="0.01"  iyz="0.0"  izz="0.016" />
       </inertial>
       <visual>
@@ -18,5 +18,5 @@
 	<origin xyz="0 0 -0.005" rpy="0 0 0"/>
 	<geometry name="shadowarm_handsupport_collision">
-	  <cylinder radius="0.06" length="0.001"/>
+	  <cylinder radius="0.0675" length="0.006"/>
 	</geometry>
       </collision>
@@ -32,6 +32,6 @@
       <axis xyz="0 0 -1" />
       <limit lower="-${M_PI/2}" upper="${M_PI/2}"
-      effort="1000.0" velocity="10.0"/>
-      <dynamics damping="30.0"/>
+      effort="30" velocity="1.0"/>
+      <dynamics damping="5.5"/>
     </joint>
     <xacro:shadowarm_handsupport_motor_transmission />

File: sr_description/arm/xacro/hand_support/shadowarm_handsupport_muscle.urdf.xacro (robot description, xacro)
@@ -6,5 +6,5 @@
 	<origin xyz="0 0 0" rpy="0 0 0" />
 	<mass value="0.75" />
-	<inertia  ixx="1.0" ixy="0.0"  ixz="0.0"  iyy="0.0"  iyz="0.0"  izz="0.0" />
+	<inertia  ixx="0.01" ixy="0.0"  ixz="0.0"  iyy="0.01"  iyz="0.0"  izz="0.016" />
       </inertial>
       <visual>
@@ -18,5 +18,5 @@
 	<origin xyz="0 0 0" rpy="0 0 0"/>
 	<geometry name="shadowarm_handsupport_collision">
-	  <cylinder radius="0.06" length="0.001"/>
+	  <cylinder radius="0.07" length="0.006"/>
 	</geometry>
       </collision>
@@ -32,6 +32,6 @@
       <axis xyz="0 0 -1" />
       <limit lower="-${M_PI/2}" upper="${M_PI/2}"
-      effort="1000.0" velocity="10.0"/>
-      <dynamics damping="20.0"/>
+      effort="30" velocity="1.0"/>
+      <dynamics damping="5.5"/>
     </joint>
     <xacro:shadowarm_handsupport_muscle_transmission />

File: sr_description/arm/xacro/lower_arm/shadowarm_lowerarm.urdf.xacro (robot description, xacro)
@@ -3,23 +3,22 @@
   <xacro:macro name="shadowarm_lowerarm" params="parent">
     <link name="shadowarm_lowerarm">
-      <inertial>
-	<origin xyz="0 0 0" rpy="0 0 0" />
-	<mass value="0.5" />
-	<inertia  ixx="0.1" ixy="0.0"  ixz="0.0"  iyy="0.1"  iyz="0.0"
-	izz="0.0" />
-      </inertial>
-      <visual>
-	<origin xyz="0.03 0 0.036" rpy="0 0 0" />
-	<geometry name="shadowarm_visual">
-          <mesh filename="package://sr_description/arm/model/elbow_flex.dae" scale="0.001 0.001 0.001" />
-        </geometry>
-        <material name="Grey" />
-      </visual>
-      <collision>
-	<origin xyz="0.03 0 0.036" rpy="0 0 0" />
-	<geometry name="shadowarm_collision_geom">
-          <mesh filename="package://sr_description/arm/model/elbow_flex.dae" scale="0.001 0.001 0.001" />
-        </geometry>
-      </collision>
+	<inertial>
+	  <origin xyz="0.08 0 0.0625" rpy="0 0 0" />
+	  <mass value="1.7" />
+	  <inertia  ixx="0.01" ixy="0.0"  ixz="0.0"  iyy="0.01"  iyz="0.0"  izz="0.01" />
+	</inertial>
+	<visual>
+	  <origin xyz="0.03 0 0.036" rpy="0 0 0"/>
+	  <geometry name="shadowarm_lowerarm_visual">
+	    <mesh filename="package://sr_description/arm/model/elbow_flex.dae" scale="0.001 0.001 0.001" />
+	  </geometry>
+	  <material name="Grey" />
+	</visual>
+	<collision>
+	  <origin xyz="0.08 0 0.0625" rpy="0 0 0"/>
+	  <geometry name="shadowarm_lowerarm_collision">
+	    <box size="0.06 0.08 0.1"/>
+	  </geometry>
+	</collision>
     </link>
     <gazebo reference="shadowarm_lowerarm">
@@ -32,6 +31,7 @@
       <origin xyz="0 0 0.369" rpy="0 0 0" />
       <axis xyz="0 -1 0" />
-      <limit lower="0.52" upper="2.09439510239" effort="1000.0" velocity="10.0"/>
-      <dynamics damping="20.0"/>
+      <limit lower="0.52" upper="2.09439510239"
+      effort="50" velocity="1.0"/>
+      <dynamics damping="5.5"/>
     </joint>
     <xacro:shadowarm_lowerarm_transmission />

File: sr_description/arm/xacro/trunk/shadowarm_trunk.urdf.xacro (robot description, xacro)
@@ -3,27 +3,27 @@
   <xacro:macro name="shadowarm_trunk" params="parent">
     <link name="shadowarm_trunk">
-      <inertial>
-        <origin xyz="0 0 0.0" rpy="0 0 0" />
-        <mass value="0.5" />
-        <inertia  ixx="0.1" ixy="0.0"  ixz="0.0"  iyy="0.1"  iyz="0.0" izz="0.0" />
-      </inertial>
-      <visual>
-	<origin xyz="0 0 0.005" rpy="0 0 0" />
-	<geometry name="shadowarm_visual">
-          <mesh filename="package://sr_description/arm/model/arm_trunk.dae" scale="0.001 0.001 0.001" />
-        </geometry>
-        <material name="Grey" />
-      </visual>
-      <collision>
-	<origin xyz="0 0 0.005" rpy="0 0 0" />
-	<geometry name="shadowarm_collision_geom">
-          <mesh filename="package://sr_description/arm/model/arm_trunk.dae" scale="0.001 0.001 0.001" />
-        </geometry>
-      </collision>
-    </link>
-    <gazebo reference="shadowarm_trunk">
-      <material>LightGrey</material>
-      <selfCollide>false</selfCollide>
-    </gazebo>
+	<inertial>
+	  <origin xyz="0 0 0.26525" rpy="0 0 0" />
+	  <mass value="10" />
+	  <inertia  ixx="0.15" ixy="0.0"  ixz="0.0"  iyy="0.15"  iyz="0.0"  izz="0.02" />
+	</inertial>
+	<visual>
+	  <origin xyz="0 0 0.005" rpy="0 0 0" />
+	  <geometry name="shadowarm_trunk_visual">
+	    <mesh filename="package://sr_description/arm/model/arm_trunk.dae" scale="0.001 0.001 0.001" />
+	  </geometry>
+	  <material name="Grey" />
+	</visual>
+	<collision>
+	  <origin xyz="0 0.02 0.30" rpy="0 0 0"/>
+	  <geometry name="shadowarm_trunk_collision">
+	    <box size="0.170 0.170 0.580"/>
+	  </geometry>
+	</collision>
+      </link>
+      <gazebo reference="shadowarm_trunk">
+	<material>LightGrey</material>
+	<selfCollide>false</selfCollide>
+      </gazebo>
     <joint name="ShoulderJRotate" type="revolute">
       <parent link="${parent}"/>
@@ -32,6 +32,6 @@
       <axis xyz="0 0 1" />
       <limit lower="-${M_PI/4}" upper="${M_PI/2}"
-      effort="1000.0" velocity="10.0"/>
-      <dynamics damping="30.0"/>
+      effort="70" velocity="1.0"/>
+      <dynamics damping="5.5"/>
     </joint>
     <xacro:shadowarm_trunk_transmission />

File: sr_description/arm/xacro/upper_arm/shadowarm_upperarm.urdf.xacro (robot description, xacro)
@@ -4,20 +4,20 @@
     <link name="shadowarm_upperarm">
       <inertial>
-        <origin xyz="0 0 0.0" rpy="0 0 0" />
-        <mass value="0.5" />
-        <inertia  ixx="0.1" ixy="0.0"  ixz="0.0"  iyy="0.1"  iyz="0.0" izz="0.0" />
+	<origin xyz="0 0 0.1845" rpy="0 0 0" />
+	<mass value="2" />
+	<inertia  ixx="0.4" ixy="0.0"  ixz="0.0"  iyy="0.4"  iyz="0.0"  izz="0.05" />
       </inertial>
       <visual>
 	<origin xyz="0 0.067 0" rpy="0 0 0" />
-	<geometry name="shadowarm_visual">
-          <mesh filename="package://sr_description/arm/model/upper_arm.dae" scale="0.001 0.001 0.001" />
-        </geometry>
-        <material name="Grey" />
+	<geometry name="shadowarm_upperarm_visual">
+	  <mesh filename="package://sr_description/arm/model/upper_arm.dae" scale="0.001 0.001 0.001" />
+	</geometry>
+	<material name="Grey" />
       </visual>
       <collision>
-	<origin xyz="0 0.067 0" rpy="0 0 0" />
-	<geometry name="shadowarm_collision_geom">
-          <mesh filename="package://sr_description/arm/model/upper_arm.dae" scale="0.001 0.001 0.001" />
-        </geometry>
+	<origin xyz="0 0 0.16" rpy="0 -${M_PI} 0"/>
+	<geometry name="shadowarm_upperarm_collision">
+	  <box size="0.170 0.133 0.470"/>
+	</geometry>
       </collision>
     </link>
@@ -31,6 +31,6 @@
       <origin xyz="0 -0.134 0.5305" rpy="0 -${M_PI} 0.0" /> <!-- yaw=-0.026 -->
       <axis xyz="0 -1 0" />
-      <limit lower="0" upper="${M_PI/2}" effort="1000.0" velocity="10.0"/>
-      <dynamics damping="30.0"/>
+      <limit lower="0" upper="${M_PI/2}" effort="100" velocity="1.0"/>
+      <dynamics damping="5.3"/>
     </joint>
     <xacro:shadowarm_upperarm_transmission />

File: sr_description/hand/xacro/finger/biotac/biotac.urdf.xacro (robot description, xacro)
@@ -11,11 +11,11 @@
       <inertial>
         <origin xyz="0 0 0.0125" rpy="0 0 0" />
-        <mass value="0.012" />
-        <inertia  ixx="0.1" ixy="0.0"  ixz="0.0"  iyy="0.1"  iyz="0.0" izz="0.01" />
+        <mass value="0.016" />
+	    <inertia ixx="0.002" ixy="0.0" ixz="0.0" iyy="0.002" iyz="0.0" izz="0.0002" />
       </inertial>
       <visual>
         <origin xyz="0 0 0" rpy="0 0 1.571" />
         <geometry name="${link_prefix}adapter_visual">
-          <mesh filename="package://sr_description/hand/model/biotacs/biotac_decimated.dae" scale="0.001 0.001 0.001" />
+          <mesh filename="package://sr_description/hand/model/biotacs/biotac_finger_adapter.dae" scale="1 1 1" />
         </geometry>
         <material name="LightGrey" />
@@ -49,7 +49,6 @@
       <origin xyz="0 0 0.045" rpy="0 0 0" />
       <axis xyz="1 0 0" />
-      <limit lower="0" upper="${M_PI/2}" effort="1000.0"
-      velocity="10.0" />
-      <dynamics damping="10.0"/>
+      <limit lower="0" upper="${M_PI/2}" effort="30" velocity="1.0"/>
+      <dynamics damping="0.1"/>
     </joint>
     <link name="${link_prefix}_J1_dummy">
@@ -57,5 +56,5 @@
         <origin xyz="0 0 0" rpy="0 0 0" />
         <mass value="0.01" />
-        <inertia  ixx="0.1" ixy="0.0"  ixz="0.0"  iyy="0.1"  iyz="0.0" izz="0.01" />
+        <inertia ixx="0.0007" ixy="0.0" ixz="0.0" iyy="0.0007" iyz="0.0" izz="0.00010" />
       </inertial>
     </link>
@@ -65,6 +64,6 @@
       <origin xyz="0 0 0.02" rpy="0 0 0" />
       <axis xyz="1 0 0" />
-      <limit lower="${20*M_PI/180}" upper="${20.1*M_PI/180}" effort="1000.0" velocity="10.0" />
-      <dynamics damping="10.0"/>
+      <limit lower="${20*M_PI/180}" upper="${20.1*M_PI/180}" effort="10" velocity="1.0"/>
+      <dynamics damping="0.1"/>
     </joint>
     <xacro:middle_transmission />
@@ -72,6 +71,6 @@
       <inertial>
         <origin xyz="0 0 0" rpy="0 0 0" />
-        <mass value="0.10" />
-        <inertia  ixx="0.1" ixy="0.0"  ixz="0.0"  iyy="0.1"  iyz="0.0" izz="0.01" />
+        <mass value="0.01" />
+        <inertia ixx="0.0007" ixy="0.0" ixz="0.0" iyy="0.0007" iyz="0.0" izz="0.00010" />
       </inertial>
       <visual>
@@ -118,5 +117,5 @@
        <mass value="0.001" />
        <origin xyz="0 0 0" rpy="0 0 0" />
-       <inertia  ixx="1" ixy="0"  ixz="0"  iyy="1"  iyz="0" izz="1" />
+       <inertia ixx="0" ixy="0" ixz="0" iyy="0" iyz="0" izz="0" />
       </inertial>
       <visual>

File: sr_description/hand/xacro/finger/biotac/edc_muscle_biotac.urdf.xacro (robot description, xacro)
@@ -11,11 +11,11 @@
       <inertial>
         <origin xyz="0 0 0.0125" rpy="0 0 0" />
-        <mass value="0.012" />
-        <inertia  ixx="0.1" ixy="0.0"  ixz="0.0"  iyy="0.1"  iyz="0.0" izz="0.01" />
+        <mass value="0.016" />
+	    <inertia ixx="0.002" ixy="0.0" ixz="0.0" iyy="0.002" iyz="0.0" izz="0.0002" />
       </inertial>
       <visual>
         <origin xyz="0 0 0" rpy="0 0 1.571" />
         <geometry name="${link_prefix}adapter_visual">
-          <mesh filename="package://sr_description/hand/model/biotacs/F2_biotac_adapter.stl" scale="0.001 0.001 0.001" />
+          <mesh filename="package://sr_description/hand/model/biotacs/biotac_finger_adapter.dae" scale="1 1 1" />
         </geometry>
         <material name="LightGrey" />
@@ -49,7 +49,6 @@
       <origin xyz="0 0 0.045" rpy="0 0 0" />
       <axis xyz="1 0 0" />
-      <limit lower="0" upper="${M_PI/2}" effort="1000.0"
-      velocity="10.0" />
-      <dynamics damping="10.0"/>
+      <limit lower="0" upper="${M_PI/2}" effort="30" velocity="1.0"/>
+      <dynamics damping="0.1"/>
     </joint>
     <link name="${link_prefix}_J1_dummy">
@@ -57,5 +56,5 @@
         <origin xyz="0 0 0" rpy="0 0 0" />
         <mass value="0.01" />
-        <inertia  ixx="0.1" ixy="0.0"  ixz="0.0"  iyy="0.1"  iyz="0.0" izz="0.01" />
+        <inertia ixx="0.0007" ixy="0.0" ixz="0.0" iyy="0.0007" iyz="0.0" izz="0.00010" />
       </inertial>
     </link>
@@ -65,6 +64,6 @@
       <origin xyz="0 0 0.02" rpy="0 0 0" />
       <axis xyz="1 0 0" />
-      <limit lower="${20*M_PI/180}" upper="${20.1*M_PI/180}" effort="1000.0" velocity="10.0" />
-      <dynamics damping="10.0"/>
+      <limit lower="${20*M_PI/180}" upper="${20.1*M_PI/180}" effort="10" velocity="1.0"/>
+      <dynamics damping="0.1"/>
     </joint>
     <xacro:middle_transmission />
@@ -72,6 +71,6 @@
       <inertial>
         <origin xyz="0 0 0" rpy="0 0 0" />
-        <mass value="0.10" />
-        <inertia  ixx="0.1" ixy="0.0"  ixz="0.0"  iyy="0.1"  iyz="0.0" izz="0.01" />
+        <mass value="0.01" />
+        <inertia ixx="0.0007" ixy="0.0" ixz="0.0" iyy="0.0007" iyz="0.0" izz="0.00010" />
       </inertial>
       <visual>
@@ -118,5 +117,5 @@
        <mass value="0.001" />
        <origin xyz="0 0 0" rpy="0 0 0" />
-       <inertia  ixx="1" ixy="0"  ixz="0"  iyy="1"  iyz="0" izz="1" />
+       <inertia ixx="0" ixy="0" ixz="0" iyy="0" iyz="0" izz="0" />
       </inertial>
       <visual>

File: sr_description/hand/xacro/finger/classic_finger_ellipsoid.urdf.xacro (robot description, xacro)
@@ -4,5 +4,5 @@
   <xacro:include filename="$(find sr_description)/hand/xacro/finger/middle/middle.urdf.xacro" />
   <xacro:include filename="$(find sr_description)/hand/xacro/finger/distal/distal_ellipsoid.urdf.xacro" />
-  <xacro:macro name="finger" params="link_prefix joint_prefix parent *origin *axis">
+  <xacro:macro name="finger_ellipsoid" params="link_prefix joint_prefix parent *origin *axis">
     <xacro:knuckle link_prefix="${link_prefix}" joint_prefix="${joint_prefix}" parent="${parent}" >
       <insert_block name="origin" />
@@ -13,6 +13,6 @@
     <xacro:middle link_prefix="${link_prefix}" joint_prefix="${joint_prefix}" parent="${link_prefix}proximal" >
     </xacro:middle>
-    <xacro:distal link_prefix="${link_prefix}" joint_prefix="${joint_prefix}" parent="${link_prefix}middle" >
-    </xacro:distal>
+    <xacro:distal_ellipsoid link_prefix="${link_prefix}" joint_prefix="${joint_prefix}" parent="${link_prefix}middle" >
+    </xacro:distal_ellipsoid>
   </xacro:macro>
 </robot>

File: sr_description/hand/xacro/finger/distal/distal.urdf.xacro (robot description, xacro)
@@ -11,7 +11,7 @@
       <inertial>
 	<mass value="0.010" />
-	<origin xyz="0 0 0.013" />
-	<inertia  ixx="0.1" ixy="0.0"  ixz="0.0"  iyy="0.1"  iyz="0.0"
-	izz="0.0" />
+	<origin xyz="0 0 0.012" />
+	<inertia ixx="0.001" ixy="0.0" ixz="0.0" iyy="0.001" iyz="0.0"
+	izz="0.00025" />
       </inertial>
       <visual>
@@ -51,7 +51,6 @@
       <origin xyz="0 0 0.025" rpy="0 0 0" />
       <axis xyz="1 0 0" />
-      <limit lower="0" upper="${M_PI/2}" effort="1000.0"
-      velocity="10.0" />
-      <dynamics damping="10.0"/>
+      <limit lower="0" upper="${M_PI/2}" effort="2" velocity="1.0" />
+      <dynamics damping="0.1"/>
     </joint>
     <link name="${link_prefix}tip">

File: sr_description/hand/xacro/finger/distal/distal_biotac.urdf.xacro (robot description, xacro)
@@ -12,6 +12,6 @@
 	<mass value="0.010" />
 	<origin xyz="0 0 0.013" />
-	<inertia  ixx="0.1" ixy="0.0"  ixz="0.0"  iyy="0.1"  iyz="0.0"
-	izz="0.0" />
+	<inertia ixx="0.001" ixy="0.0" ixz="0.0" iyy="0.001" iyz="0.0"
+	izz="0.00025" />
       </inertial>
       <visual>
@@ -51,7 +51,6 @@
       <origin xyz="0 0 0.025" rpy="0 0 0" />
       <axis xyz="1 0 0" />
-      <limit lower="0.34906585" upper="0.34906585" effort="1000.0"
-      velocity="10.0" />
-      <dynamics damping="10.0"/>
+      <limit lower="0" upper="${M_PI/2}" effort="2" velocity="1.0" />
+      <dynamics damping="0.1"/>
     </joint>
 <!--

File: sr_description/hand/xacro/finger/distal/distal_ellipsoid.urdf.xacro (robot description, xacro)
@@ -7,11 +7,11 @@
        xmlns:geom="http://playerstage.sourceforge.net/gazebo/xmlschema/#geom">
   <xacro:include filename="$(find sr_description)/hand/xacro/finger/distal/distal.transmission.xacro" />
-  <xacro:macro name="distal" params="link_prefix joint_prefix parent">
+  <xacro:macro name="distal_ellipsoid" params="link_prefix joint_prefix parent">
     <link name="${link_prefix}distal">
       <inertial>
 	<mass value="0.010" />
 	<origin xyz="0 0 0.013" />
-	<inertia  ixx="0.1" ixy="0.0"  ixz="0.0"  iyy="0.1"  iyz="0.0"
-		  izz="0.0" />
+	<inertia ixx="0.001" ixy="0.0" ixz="0.0" iyy="0.001" iyz="0.0"
+	izz="0.00025" />
       </inertial>
       <visual>
@@ -58,7 +58,6 @@
       <origin xyz="0 0 0.025" rpy="0 0 0" />
       <axis xyz="1 0 0" />
-      <limit lower="0" upper="${M_PI/2}" effort="1000.0"
-	     velocity="10.0" />
-      <dynamics damping="10.0"/>
+      <limit lower="0" upper="${M_PI/2}" effort="2" velocity="1.0" />
+      <dynamics damping="0.1"/>
     </joint>
     <link name="${link_prefix}tip">

File: sr_description/hand/xacro/finger/knuckle/edc_muscle_knuckle.urdf.xacro (robot description, xacro)
@@ -12,7 +12,6 @@
 	<origin xyz="0 0 0" rpy="0 0 0" />
 	<!--<insert_block name="origin" /> -->
-	<mass value="0.008" />
-	<inertia  ixx="0.0" ixy="0.0"  ixz="0.0"  iyy="0.1"  iyz="0.0"
-	izz="0.0" />
+	<mass value="0.08" />
+	<inertia ixx="0.0026" ixy="0.0" ixz="0.0" iyy="0.0026" iyz="0.0" izz="0.0032" />
       </inertial>
       <visual>
@@ -24,7 +23,7 @@
       </visual>
       <collision>
-	<origin xyz="0 0 0" rpy="0 0 0" />
+	<origin xyz="0 0 0" rpy="0 1.5708 0" />
 	<geometry name="${link_prefix}knuckle_collision_geom">
-	  <box size="0.005 0.005 0.005" />
+	  <cylinder radius="0.007" length="0.014" />
 	</geometry>
       </collision>
@@ -52,7 +51,7 @@
       <insert_block name="origin" />
       <insert_block name="axis"/>
-      <limit lower="-0.43633231299858238" upper="0.43633231299858238"
-      effort="1000.0" velocity="10.0"/>
-      <dynamics damping="10.0"/>
+      <limit lower="${-20/180*M_PI}" upper="${20/180*M_PI}"
+      effort="2" velocity="1.0"/>
+      <dynamics damping="0.1"/>
     </joint>
     <xacro:knuckle_transmission />

File: sr_description/hand/xacro/finger/knuckle/knuckle.urdf.xacro (robot description, xacro)
@@ -12,7 +12,6 @@
 	<origin xyz="0 0 0" rpy="0 0 0" />
 	<!--<insert_block name="origin" /> -->
-	<mass value="0.008" />
-	<inertia  ixx="0.0" ixy="0.0"  ixz="0.0"  iyy="0.1"  iyz="0.0"
-	izz="0.0" />
+	<mass value="0.08" />
+	<inertia ixx="0.0026" ixy="0.0" ixz="0.0" iyy="0.0026" iyz="0.0" izz="0.0032" />
       </inertial>
       <visual>
@@ -24,7 +23,7 @@
       </visual>
       <collision>
-	<origin xyz="0 0 0" rpy="0 0 0" />
+	<origin xyz="0 0 0" rpy="0 1.5708 0" />
 	<geometry name="${link_prefix}knuckle_collision_geom">
-	  <box size="0.005 0.005 0.005" />
+	  <cylinder radius="0.007" length="0.014" />
 	</geometry>
       </collision>
@@ -52,7 +51,7 @@
       <insert_block name="origin" />
       <insert_block name="axis"/>
-      <limit lower="-0.3491" upper="0.3491"
-      effort="1000.0" velocity="10.0"/>
-      <dynamics damping="10.0"/>
+      <limit lower="${-20/180*M_PI}" upper="${20/180*M_PI}"
+      effort="2" velocity="1.0"/>
+      <dynamics damping="0.1"/>
     </joint>
     <xacro:knuckle_transmission />

File: sr_description/hand/xacro/finger/lfmetacarpal/edc_muscle_lfmetacarpal.urdf.xacro (robot description, xacro)
@@ -21,6 +21,6 @@
       <inertial>
         <origin xyz="0 0 0.04" rpy="0 0 0" />
-	    <mass value="0.075" />
-	    <inertia  ixx="0.1" ixy="0.0"  ixz="0.0"  iyy="0.1"  iyz="0.0" izz="0.1" />
+	    <mass value="0.030" />
+	    <inertia ixx="0.00545" ixy="0.0" ixz="0.0" iyy="0.0056352" iyz="0.0" izz="0.0004272" />
       </inertial>
       <visual>
@@ -32,7 +32,7 @@
       </visual>
       <collision>
-          <origin xyz="0 0 0.04" rpy="0 0 0" />
+        <origin xyz="0 0 0.038" rpy="0 0 0" />
         <geometry name="lfmetacarpal_collision_geom">
-          <box size="0.008 0.008 0.03" />
+          <box size="0.018 0.024 0.048" />
         </geometry>
       </collision>
@@ -52,4 +52,5 @@
         </plugin>
       </sensor>
+      <selfCollide>true</selfCollide>
       <material>LightGrey</material>
     </gazebo>
@@ -59,7 +60,7 @@
       <origin xyz="${reflect*-0.033} 0 0.02071" rpy="0 0 0" />
       <axis xyz="0.573576436 0 ${reflect*0.819152044}" />
-      <limit lower="0" upper="0.69813170079773179" effort="1000.0"
-      velocity="10.0" />
-      <dynamics damping="10.0"/>
+      <limit lower="0" upper="${45/180*M_PI}" effort="2"
+      velocity="1.0" />
+      <dynamics damping="0.1"/>
     </joint>
     <xacro:lfmetacarpal_transmission />
