Commit message: Rebase from 'upstream'

File: sr_description/hand/xacro/finger/lfmetacarpal/lfmetacarpal.urdf.xacro (robot description, xacro)
@@ -21,6 +21,6 @@
       <inertial>
         <origin xyz="0 0 0.04" rpy="0 0 0" />
-	    <mass value="0.075" />
-	    <inertia  ixx="0.1" ixy="0.0"  ixz="0.0"  iyy="0.1"  iyz="0.0" izz="0.1" />
+	    <mass value="0.030" />
+	    <inertia ixx="0.00545" ixy="0.0" ixz="0.0" iyy="0.0056352" iyz="0.0" izz="0.0004272" />
       </inertial>
       <visual>
@@ -32,7 +32,7 @@
       </visual>
       <collision>
-          <origin xyz="0 0 0.04" rpy="0 0 0" />
+        <origin xyz="0 0 0.038" rpy="0 0 0" />
         <geometry name="lfmetacarpal_collision_geom">
-          <box size="0.008 0.008 0.03" />
+          <box size="0.018 0.024 0.040" />
         </geometry>
       </collision>
@@ -52,4 +52,5 @@
         </plugin>
       </sensor>
+      <selfCollide>true</selfCollide>
       <material>LightGrey</material>
     </gazebo>
@@ -59,7 +60,7 @@
       <origin xyz="${reflect*-0.033} 0 0.02071" rpy="0 0 0" />
       <axis xyz="0.573576436 0 ${reflect*0.819152044}" />
-      <limit lower="0" upper="0.785398163" effort="1000.0"
-      velocity="10.0" />
-      <dynamics damping="10.0"/>
+      <limit lower="0" upper="${45/180*M_PI}" effort="2"
+      velocity="1.0" />
+      <dynamics damping="0.1"/>
     </joint>
     <xacro:lfmetacarpal_transmission />

File: sr_description/hand/xacro/finger/little_finger_ellipsoid.urdf.xacro (robot description, xacro)
@@ -6,71 +6,21 @@
        xmlns:body="http://playerstage.sourceforge.net/gazebo/xmlschema/#body"
        xmlns:geom="http://playerstage.sourceforge.net/gazebo/xmlschema/#geom">
-  <xacro:include filename="$(find sr_description)/hand/xacro/finger/knuckle/knuckle.urdf.xacro" />
-  <xacro:include filename="$(find sr_description)/hand/xacro/finger/proximal/proximal.urdf.xacro" />
-  <xacro:include filename="$(find sr_description)/hand/xacro/finger/middle/middle.urdf.xacro" />
-  <xacro:include filename="$(find sr_description)/hand/xacro/finger/distal/distal_ellipsoid.urdf.xacro" />
   <xacro:include filename="$(find sr_description)/hand/xacro/finger/lfmetacarpal/lfmetacarpal.urdf.xacro" />
+  <xacro:include filename="$(find sr_description)/hand/xacro/finger/classic_finger_ellipsoid.urdf.xacro" />
+  <!-- Right Handed -->
   <xacro:macro name="little_finger" params="link_prefix joint_prefix parent">
-    <xacro:lfmetacarpal parent="${parent}" >
-    </xacro:lfmetacarpal>
-    <link name="lfknuckle">
-      <inertial>
-	<origin xyz="0 0 0.06579" rpy="0 0 0" />
-	<mass value="0.008" />
-	<inertia  ixx="0.1" ixy="0.0"  ixz="0.0"  iyy="0.1"  iyz="0.0"
-	izz="0.1" />
-      </inertial>
-      <visual>
-	<origin xyz="0 0 0" rpy="0 0 0" />
-	<geometry name="knuckle_visual">
-      <mesh filename="package://sr_description/hand/model/knuckle.dae" scale="0.001 0.001 0.001" />
-      </geometry>
-      <material name="LightGrey" />
-      </visual>
-      <collision>
-	<origin xyz="0 0 0" rpy="0 0 0" />
-	<geometry name="knuckle_collision_geom">
-	  <box size="0.005 0.005 0.005" />
-	</geometry>
-      </collision>
-    </link>
-    <gazebo reference="lfknuckle">
-      <sensor type="contact" name="lfknuckle_contact" >
-        <always_on>1</always_on>
-        <update_rate>1000.0</update_rate>
-        <contact>
-          <collision>lfknuckle_collision</collision>
-          <topic>lfknuckle_collision</topic>
-        </contact>
-        <plugin name="lfknuckle_gazebo_ros_bumper_controller" filename="libgazebo_ros_bumper.so">
-          <updateRate>100.0</updateRate>
-	  <frameName>lfknuckle</frameName>
-	  <bumperTopicName>contacts/lf/knuckle</bumperTopicName>
-        </plugin>
-      </sensor>
-      <material>Gazebo/Grey</material>
-    </gazebo>
-    <joint name="LFJ4" type="revolute">
-      <parent link="lfmetacarpal"/>
-      <child link="lfknuckle"/>
+    <xacro:lfmetacarpal parent="${parent}" />
+    <xacro:finger_ellipsoid link_prefix="${link_prefix}" joint_prefix="${joint_prefix}" parent="lfmetacarpal">
       <origin xyz="0 0 0.06579" rpy="0 0 0" />
       <axis xyz="0 1 0" />
-      <limit lower="-0.3491" upper="0.3491"
-      effort="1000.0" velocity="10.0"/>
-      <dynamics damping="10.0"/>
-    </joint>
-    <transmission type="sr_mechanism_model/SimpleTransmission" name="lfknuckle_transmission">
-      <actuator name="LFJ4" />
-      <joint name="LFJ4" />
-      <mechanicalReduction>1</mechanicalReduction>
-      <motorTorqueConstant>1</motorTorqueConstant>
-      <pulsesPerRevolution>90000</pulsesPerRevolution>
-    </transmission>
-    <xacro:proximal link_prefix="${link_prefix}" joint_prefix="${joint_prefix}" parent="${link_prefix}knuckle" >
-    </xacro:proximal>
-    <xacro:middle link_prefix="${link_prefix}" joint_prefix="${joint_prefix}" parent="${link_prefix}proximal" >
-    </xacro:middle>
-    <xacro:distal link_prefix="${link_prefix}" joint_prefix="${joint_prefix}" parent="${link_prefix}middle" >
-    </xacro:distal>
+    </xacro:finger_ellipsoid>
+  </xacro:macro>
+  <!-- Left Handed -->
+  <xacro:macro name="little_finger_left" params="link_prefix joint_prefix parent">
+    <xacro:lfmetacarpal_left parent="${parent}" />
+    <xacro:finger_ellipsoid link_prefix="${link_prefix}" joint_prefix="${joint_prefix}" parent="lfmetacarpal">
+      <origin xyz="0 0 0.06579" rpy="0 0 0" />
+      <axis xyz="0 -1 0" />
+    </xacro:finger_ellipsoid>
   </xacro:macro>
 </robot>

File: sr_description/hand/xacro/finger/middle/middle.urdf.xacro (robot description, xacro)
@@ -11,7 +11,6 @@
       <inertial>
 	<origin xyz="0 0 0.0125" rpy="0 0 0" />
-	<mass value="0.012" />
-	<inertia  ixx="0.1" ixy="0.0"  ixz="0.0"  iyy="0.1"  iyz="0.0"
-	izz="0.0" />
+	<mass value="0.020" />
+	<inertia ixx="0.002" ixy="0.0" ixz="0.0" iyy="0.002" iyz="0.0" izz="0.0002" />
       </inertial>
       <visual>
@@ -22,9 +21,21 @@
       <material name="Grey" />
       </visual>
+    <collision>
+        <origin xyz="0 0 0.0125" rpy="0 0 0 " />
+        <geometry name="${link_prefix}middle_collision_geom">
+          <cylinder radius="0.007" length="0.025" />
+        </geometry>
+      </collision>
       <collision>
-	<origin xyz="0 0 0.0125" rpy="0 0 0" />
-	<geometry name="${link_prefix}middle_collision_geom">
-	  <box size="0.008 0.008 0.015" />
-	</geometry>
+        <origin xyz="0 0 0.0" rpy="0 0 0 " />
+        <geometry>
+          <sphere radius="0.007" />
+        </geometry>
+      </collision>
+      <collision>
+        <origin xyz="0 0 0.025" rpy="0 0 0 " />
+        <geometry>
+          <sphere radius="0.007" />
+        </geometry>
       </collision>
     </link>
@@ -43,4 +54,5 @@
         </plugin>
       </sensor>
+       <selfCollide>true</selfCollide>
       <material>LightGrey</material>
     </gazebo>
@@ -50,7 +62,7 @@
       <origin xyz="0 0 0.045" rpy="0 0 0" />
       <axis xyz="1 0 0" />
-      <limit lower="0" upper="${M_PI/2}" effort="1000.0"
-      velocity="10.0" />
-      <dynamics damping="10.0"/>
+      <limit lower="0" upper="${M_PI/2}" effort="2"
+      velocity="1.0" />
+      <dynamics damping="0.1"/>
     </joint>
     <xacro:middle_transmission />

File: sr_description/hand/xacro/finger/proximal/edc_muscle_proximal.urdf.xacro (robot description, xacro)
@@ -10,8 +10,7 @@
     <link name="${link_prefix}proximal">
       <inertial>
-	<mass value="0.014" />
-	<origin xyz="0 0 0.0225" />
-	<inertia  ixx="0.1" ixy="0.0"  ixz="0.0"  iyy="0.1"  iyz="0.0"
-	izz="0.0" />
+	    <mass value="0.030" />
+        <origin xyz="0 0 0.0225" />
+        <inertia ixx="0.003" ixy="0.0" ixz="0.0" iyy="0.003" iyz="0.0" izz="0.0003" />
       </inertial>
       <visual>
@@ -23,8 +22,8 @@
       </visual>
       <collision>
-	<origin xyz="0 0 0.025" rpy="0 0 0 " />
-	<geometry name="proximal_collision_geom">
-	  <box size="0.008 0.008 0.04" />
-	</geometry>
+        <origin xyz="0 0 0.025" rpy="0 0 0 " />
+        <geometry name="${link_prefix}proximal_collision_geom">
+          <cylinder radius="0.007" length="0.040" />
+        </geometry>
       </collision>
     </link>
@@ -43,4 +42,5 @@
         </plugin>
       </sensor>
+      <selfCollide>true</selfCollide>
       <material>LightGrey</material>
     </gazebo>
@@ -50,7 +50,7 @@
       <origin xyz="0 0 0" rpy="0 0 0" />
       <axis xyz="1 0 0" />
-      <limit lower="0" upper="${M_PI/2}" effort="1000.0"
-      velocity="10.0"/>
-      <dynamics damping="10.0"/>
+      <limit lower="0" upper="${M_PI/2}" effort="2"
+      velocity="1.0"/>
+      <dynamics damping="0.1"/>
     </joint>
     <xacro:proximal_transmission />

File: sr_description/hand/xacro/finger/proximal/proximal.urdf.xacro (robot description, xacro)
@@ -10,21 +10,20 @@
     <link name="${link_prefix}proximal">
       <inertial>
-	<mass value="0.014" />
-	<origin xyz="0 0 0.0225" />
-	<inertia  ixx="0.1" ixy="0.0"  ixz="0.0"  iyy="0.1"  iyz="0.0"
-	izz="0.0" />
+        <mass value="0.030" />
+        <origin xyz="0 0 0.0225" />
+        <inertia ixx="0.003" ixy="0.0" ixz="0.0" iyy="0.003" iyz="0.0" izz="0.0003" />
       </inertial>
       <visual>
-	<origin xyz="0 0 0" rpy="0 0 0" />
-	<geometry name="proximal_visual">
-      <mesh filename="package://sr_description/hand/model/F3.dae" scale="0.001 0.001 0.001" />
-      </geometry>
-      <material name="Grey" />
+      <origin xyz="0 0 0" rpy="0 0 0" />
+        <geometry name="${link_prefix}proximal_visual">
+          <mesh filename="package://sr_description/hand/model/F3.dae" scale="0.001 0.001 0.001" />
+        </geometry>
+        <material name="Grey" />
       </visual>
       <collision>
-	<origin xyz="0 0 0.025" rpy="0 0 0 " />
-	<geometry name="proximal_collision_geom">
-	  <box size="0.008 0.008 0.04" />
-	</geometry>
+        <origin xyz="0 0 0.025" rpy="0 0 0 " />
+        <geometry name="${link_prefix}proximal_collision_geom">
+          <cylinder radius="0.007" length="0.040" />
+        </geometry>
       </collision>
     </link>
@@ -43,4 +42,5 @@
         </plugin>
       </sensor>
+       <selfCollide>true</selfCollide>
       <material>LightGrey</material>
     </gazebo>
@@ -50,7 +50,7 @@
       <origin xyz="0 0 0" rpy="0 0 0" />
       <axis xyz="1 0 0" />
-      <limit lower="0" upper="${M_PI/2}" effort="1000.0"
-      velocity="10.0"/>
-      <dynamics damping="10.0"/>
+      <limit lower="0" upper="${M_PI/2}" effort="2"
+      velocity="1.0"/>
+      <dynamics damping="0.1"/>
     </joint>
     <xacro:proximal_transmission />
